File: hardware/rev2026/picoemp-rev2026.kicad_sch (KiCad schematic)
At the start: 47 parts, among them J1 Header 7, J2 1x2_Pin_Header, J3 BG306-02-A-2-0400-L-G, J4 Header 2, J5 Header 4, J6 EDGE-SMA, Q1 LDA111STR, Q2 RGT16BM65DTL, Q3 AO3422, Q4 AO3422, SW1 KSC741J LFS, SW2 KSC741J LFS, SW3 TL3301AF160QJ, T1 ATB322524, T2 ATB322524, U1 SC0915

Commit message: Assign resolvable footprints to all but switches, headers and J3
Fills in every symbol whose footprint was empty, a bare manufacturer
part number, a HandSolder-pad variant string, or the corrupt Altium
SamacSys path, per the Rev-2026 design spec section 6.1. D1/D3/D4/D5
use the project-local picoemp:D_SOD-123FL (Task 6) rather than KiCad's
stock D_SOD-123F, whose land is 0.3mm narrower than the correct part.

SW1-3 and J3 stay empty (Task 8/9/11 own them); J1/J4/J5 keep their
wrong-pitch Altium header footprints since they get renamed to
P1/P2/P3 with 2.54mm footprints in Task 8.
Parts:
- C1, C2: footprint Capacitor_SMD:C_0805_2012Metric_Pad1.18x1.45mm_HandSolder -> Capacitor_SMD:C_0805_2012Metric
- C3: footprint CKG57N_2220 -> Capacitor_SMD:C_2220_5750Metric
- C5: footprint Capacitor_SMD:C_0603_1608Metric_Pad1.08x0.95mm_HandSolder -> Capacitor_SMD:C_0603_1608Metric
- D1: footprint (none) -> picoemp:D_SOD-123FL
- D2: footprint SMA -> Diode_SMD:D_SMA
- D3, D4, D5: footprint DSS13UTR -> picoemp:D_SOD-123FL
- D7: footprint SOD323 -> Diode_SMD:D_SOD-323F
- J2: footprint Connector_PinHeader_1.27mm:PinHeader_1x02_P1.27mm_Vertical -> Connector_JST:JST_XH_S2B-XH-A_1x02_P2.50mm_Horizontal
- LED1, LED2, LED3: footprint LED_SMD:LED_0603_1608Metric_Pad1.05x0.95mm_HandSolder -> LED_SMD:LED_0603_1608Metric
- Q1: footprint C__Users_colin_Documents_AltiumLL_SamacSys.PcbLib:SOP254P952X470-6N -> picoemp:SOP-6_LDA111
- Q2: footprint (none) -> Package_TO_SOT_SMD:TO-252-3_TabPin2
- Q3, Q4: footprint (none) -> Package_TO_SOT_SMD:SOT-23
- R1: footprint Resistor_SMD:R_2010_5025Metric_Pad1.40x2.65mm_HandSolder -> Resistor_SMD:R_2010_5025Metric
- R10, R11, R12, R13, R3, R5, R6, R7: footprint Resistor_SMD:R_0603_1608Metric_Pad0.98x0.95mm_HandSolder -> Resistor_SMD:R_0603_1608Metric
- R2: footprint Resistor_SMD:R_2512_6332Metric_Pad1.40x3.35mm_HandSolder -> Resistor_SMD:R_2512_6332Metric
- R4, R9: footprint Resistor_SMD:R_0805_2012Metric_Pad1.20x1.40mm_HandSolder -> Resistor_SMD:R_0805_2012Metric
- T1, T2: footprint ATB322524 -> picoemp:ATB322524
Changed lines of the file:
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@@
 			)
 		)
-		(property "Footprint" "Resistor_SMD:R_0603_1608Metric_Pad0.98x0.95mm_HandSolder"
+		(property "Footprint" "Resistor_SMD:R_0603_1608Metric"
 			(at 83.82 132.08 0)
 			(hide yes)
@@
 			)
 		)
-		(property "Footprint" "Resistor_SMD:R_0603_1608Metric_Pad0.98x0.95mm_HandSolder"
+		(property "Footprint" "Resistor_SMD:R_0603_1608Metric"
 			(at 223.52 114.3 0)
 			(hide yes)
@@
 			)
 		)
-		(property "Footprint" "Capacitor_SMD:C_0603_1608Metric_Pad1.08x0.95mm_HandSolder"
+		(property "Footprint" "Capacitor_SMD:C_0603_1608Metric"
 			(at 273.812 357.886 90)
 			(hide yes)
@@
 			)
 		)
-		(property "Footprint" "DSS13UTR"
+		(property "Footprint" "picoemp:D_SOD-123FL"
 			(at 185.42 315.468 90)
 			(hide yes)
@@
 			)
 		)
-		(property "Footprint" "DSS13UTR"
+		(property "Footprint" "picoemp:D_SOD-123FL"
 			(at 226.06 300.228 90)
 			(hide yes)
@@
 			)
 		)
-		(property "Footprint" "DSS13UTR"
+		(property "Footprint" "picoemp:D_SOD-123FL"
 			(at 220.98 361.188 90)
 			(hide yes)
@@
 			)
 		)
-		(property "Footprint" "Capacitor_SMD:C_0805_2012Metric_Pad1.18x1.45mm_HandSolder"
+		(property "Footprint" "Capacitor_SMD:C_0805_2012Metric"
 			(at 268.732 299.466 90)
 			(hide yes)
@@
 			)
 		)
-		(property "Footprint" "LED_SMD:LED_0603_1608Metric_Pad1.05x0.95mm_HandSolder"
+		(property "Footprint" "LED_SMD:LED_0603_1608Metric"
 			(at 228.854 119.888 90)
 			(hide yes)
@@
 			)
 		)
-		(property "Footprint" "SMA"
+		(property "Footprint" "Diode_SMD:D_SMA"
 			(at 322.58 282.448 90)
 			(hide yes)
@@
 			)
 		)
-		(property "Footprint" ""
+		(property "Footprint" "Package_TO_SOT_SMD:TO-252-3_TabPin2"
 			(at 381 292.1 0)
 			(hide yes)
@@
 			)
 		)
-		(property "Footprint" ""
+		(property "Footprint" "Package_TO_SOT_SMD:SOT-23"
 			(at 259.08 292.1 0)
 			(hide yes)
@@
 			)
 		)
-		(property "Footprint" "Resistor_SMD:R_0603_1608Metric_Pad0.98x0.95mm_HandSolder"
+		(property "Footprint" "Resistor_SMD:R_0603_1608Metric"
 			(at 350.52 335.28 0)
 			(hide yes)
@@
 			)
 		)
-		(property "Footprint" "CKG57N_2220"
+		(property "Footprint" "Capacitor_SMD:C_2220_5750Metric"
 			(at 339.852 286.766 90)
 			(hide yes)
@@
 			)
 		)
-		(property "Footprint" "Resistor_SMD:R_0603_1608Metric_Pad0.98x0.95mm_HandSolder"
+		(property "Footprint" "Resistor_SMD:R_0603_1608Metric"
 			(at 83.82 116.84 0)
 			(hide yes)
@@
 			)
 		)
-		(property "Footprint" "Capacitor_SMD:C_0805_2012Metric_Pad1.18x1.45mm_HandSolder"
+		(property "Footprint" "Capacitor_SMD:C_0805_2012Metric"
 			(at 281.432 299.466 90)
 			(hide yes)
@@
 			)
 		)
-		(property "Footprint" "LED_SMD:LED_0603_1608Metric_Pad1.05x0.95mm_HandSolder"
+		(property "Footprint" "LED_SMD:LED_0603_1608Metric"
 			(at 63.5 137.668 90)
 			(hide yes)
@@
 			)
 		)
-		(property "Footprint" "Resistor_SMD:R_0603_1608Metric_Pad0.98x0.95mm_HandSolder"
+		(property "Footprint" "Resistor_SMD:R_0603_1608Metric"
 			(at 256.54 233.68 0)
 			(hide yes)
@@
 			)
 		)
-		(property "Footprint" "ATB322524"
+		(property "Footprint" "picoemp:ATB322524"
 			(at 296.672 334.518 90)
 			(hide yes)
@@
 			)
 		)
-		(property "Footprint" "LED_SMD:LED_0603_1608Metric_Pad1.05x0.95mm_HandSolder"
+		(property "Footprint" "LED_SMD:LED_0603_1608Metric"
 			(at 63.5 122.428 90)
 			(hide yes)
@@
 			)
 		)
-		(property "Footprint" "ATB322524"
+		(property "Footprint" "picoemp:ATB322524"
 			(at 296.672 276.098 90)
 			(hide yes)
@@
 			)
 		)
-		(property "Footprint" "SOD323"
+		(property "Footprint" "Diode_SMD:D_SOD-323F"
 			(at 360.172 343.154 0)
 			(hide yes)
@@
 			)
 		)
-		(property "Footprint" ""
+		(property "Footprint" "Package_TO_SOT_SMD:SOT-23"
 			(at 259.08 355.6 0)
 			(hide yes)
@@
 			)
 		)
-		(property "Footprint" "Resistor_SMD:R_0603_1608Metric_Pad0.98x0.95mm_HandSolder"
+		(property "Footprint" "Resistor_SMD:R_0603_1608Metric"
 			(at 213.36 342.9 0)
 			(hide yes)
@@
 			)
 		)
-		(property "Footprint" "Resistor_SMD:R_2512_6332Metric_Pad1.40x3.35mm_HandSolder"
+		(property "Footprint" "Resistor_SMD:R_2512_6332Metric"
 			(at 368.3 246.38 0)
 			(hide yes)
@@
 			)
 		)
-		(property "Footprint" "Resistor_SMD:R_0603_1608Metric_Pad0.98x0.95mm_HandSolder"
+		(property "Footprint" "Resistor_SMD:R_0603_1608Metric"
 			(at 243.84 363.22 0)
 			(hide yes)
@@
 			)
 		)
-		(property "Footprint" "Resistor_SMD:R_2010_5025Metric_Pad1.40x2.65mm_HandSolder"
+		(property "Footprint" "Resistor_SMD:R_2010_5025Metric"
 			(at 353.06 228.6 0)
 			(hide yes)
@@
 			)
 		)
-		(property "Footprint" "Resistor_SMD:R_0805_2012Metric_Pad1.20x1.40mm_HandSolder"
+		(property "Footprint" "Resistor_SMD:R_0805_2012Metric"
 			(at 213.36 284.48 0)
 			(hide yes)
@@
 			)
 		)
-		(property "Footprint" "C__Users_colin_Documents_AltiumLL_SamacSys.PcbLib:SOP254P952X470-6N"
+		(property "Footprint" "picoemp:SOP-6_LDA111"
 			(at 317.5 236.22 0)
 			(hide yes)
@@
 			)
 		)
-		(property "Footprint" "Connector_PinHeader_1.27mm:PinHeader_1x02_P1.27mm_Vertical"
+		(property "Footprint" "Connector_JST:JST_XH_S2B-XH-A_1x02_P2.50mm_Horizontal"
 			(at 142.24 38.1 0)
 			(hide yes)
@@
 			)
 		)
-		(property "Footprint" "Resistor_SMD:R_0603_1608Metric_Pad0.98x0.95mm_HandSolder"
+		(property "Footprint" "Resistor_SMD:R_0603_1608Metric"
 			(at 241.3 299.72 0)
 			(hide yes)
@@
 			)
 		)
-		(property "Footprint" "Resistor_SMD:R_0805_2012Metric_Pad1.20x1.40mm_HandSolder"
+		(property "Footprint" "Resistor_SMD:R_0805_2012Metric"
 			(at 330.2 340.36 0)
 			(hide yes)
@@
 			)
 		)
-		(property "Footprint" ""
+		(property "Footprint" "picoemp:D_SOD-123FL"
 			(at 142.24 54.61 90)
 			(hide yes)
