File: hardware/rev2026/picoemp-rev2026.kicad_sch (KiCad schematic)
At the start: 53 parts, among them J1 EDGE-SMA, J2 1x2_Pin_Header, J3 MKDS 1,5/2-5.08, J4 EDGE-SMA, P1 Header 7, P2 Header 2, P3 Header 4, Q1 LDA111STR, Q2 RGT16BM65DTL, Q3 AO3422, Q4 AO3422, SW1 KSC741J LFS, SW2 KSC741J LFS, SW3 TL3301AF160QJ, T1 ATB322524, T2 ATB322524, U1 SC0915, U2 74LVC1G17

Commit message: Fix MH1-3 mounting hole symbol/footprint mismatch and restore LDA111 pin 3 NC
MH1-3 used Mechanical:MountingHole_Pad_MP (pin "MP") with footprint
MountingHole:MountingHole_3.2mm_M3_Pad_Via (pad "1"), a numbering mismatch
in both directions that produced per-hole ERC warnings/errors and left
plated copper floating at no defined potential inside the HV region.
Switched to Mechanical:MountingHole / MountingHole_3.2mm_M3, which have no
pins/pads at all (the 1551B shield is plastic, so no chassis bond is
needed).

picoemp:LDA111 was missing pin 3 entirely, even though the SOP-6 footprint
correctly has six pads (the lead exists on the package, it's just
electrically NC). Restored pin 3 as an explicit no_connect/"NC" pin,
matching the original Altium design, and added a no-connect flag at Q1 in
the schematic so ERC is explicit about the intent.

Updated the schematic's embedded lib_symbols cache to match both library
edits (kicad-cli resolves geometry from that cache, not live library
lookup). Netlist membership diff confirms only the intended changes:
MH1/MH2/MH3 contribute no netlist nodes, Q1.3 appears on its own
unconnected net, and the HV feedback chain (Q1.1-R1, Q1.2-Q2.3) is
byte-for-byte unchanged. ERC is clean (0 errors) before and after.

Added regression tests covering both fixes.
Parts:
- MH1, MH2, MH3: footprint MountingHole:MountingHole_3.2mm_M3_Pad_Via -> MountingHole:MountingHole_3.2mm_M3; symbol Mechanical:MountingHole_Pad_MP -> Mechanical:MountingHole
Connections:
- no-connect marks 26 -> 27
Changed lines of the file:
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@@
 		(at 165.1 99.06)
 	)
+	(no_connect
+		(at 317.5 241.3)
+	)
 	(wire
 		(pts
@@
 	)
 	(symbol
-		(lib_id "Mechanical:MountingHole_Pad_MP")
+		(lib_id "Mechanical:MountingHole")
 		(at 123.19 210.82 0)
 		(unit 1)
@@
 			)
 		)
-		(property "Footprint" "MountingHole:MountingHole_3.2mm_M3_Pad_Via"
+		(property "Footprint" "MountingHole:MountingHole_3.2mm_M3"
 			(at 128.27 209.153 90)
 			(hide yes)
@@
 			)
 		)
-		(property "Description" "Mounting Hole with connection as pad named MP"
+		(property "Description" "Mounting Hole without connection"
 			(at 123.19 210.82 0)
 			(hide yes)
@@
 			)
 		)
-		(pin "MP"
-		)
 		(instances
 			(project "picoemp-rev2026"
@@
 		(pin "4"
 		)
+		(pin "3"
+		)
 		(instances
 			(project "picoemp-rev2026"
@@
 	)
 	(symbol
-		(lib_id "Mechanical:MountingHole_Pad_MP")
+		(lib_id "Mechanical:MountingHole")
 		(at 123.19 195.58 0)
 		(unit 1)
@@
 			)
 		)
-		(property "Footprint" "MountingHole:MountingHole_3.2mm_M3_Pad_Via"
+		(property "Footprint" "MountingHole:MountingHole_3.2mm_M3"
 			(at 128.27 193.913 90)
 			(hide yes)
@@
 			)
 		)
-		(property "Description" "Mounting Hole with connection as pad named MP"
+		(property "Description" "Mounting Hole without connection"
 			(at 123.19 195.58 0)
 			(hide yes)
@@
 			)
 		)
-		(pin "MP"
-		)
 		(instances
 			(project "picoemp-rev2026"
@@
 	)
 	(symbol
-		(lib_id "Mechanical:MountingHole_Pad_MP")
+		(lib_id "Mechanical:MountingHole")
 		(at 123.19 226.06 0)
 		(unit 1)
@@
 			)
 		)
-		(property "Footprint" "MountingHole:MountingHole_3.2mm_M3_Pad_Via"
+		(property "Footprint" "MountingHole:MountingHole_3.2mm_M3"
 			(at 128.27 224.393 90)
 			(hide yes)
@@
 			)
 		)
-		(property "Description" "Mounting Hole with connection as pad named MP"
+		(property "Description" "Mounting Hole without connection"
 			(at 123.19 226.06 0)
 			(hide yes)
@@
 			)
 		)
-		(pin "MP"
-		)
 		(instances
