File: hardware/rev2026/picoemp-rev2026.kicad_sch (KiCad schematic)
At the start: 53 parts, among them J1 EDGE-SMA, J2 1x2_Pin_Header, J3 MKDS 1,5/2-5.08, J4 EDGE-SMA, P1 Header 7, P2 Header 2, P3 Header 4, Q1 LDA111STR, Q2 RGT16BM65DTL, Q3 AO3422, Q4 AO3422, SW1 KSC741J LFS, SW2 KSC741J LFS, SW3 TL3301AF160QJ, T1 ATB322524, T2 ATB322524, U1 SC0915, U2 74LVC1G17

Commit message: Swap J1/J4 to the TE/Linx CONSMA020.062-G edge-mount SMA
Replaces the Amphenol 132289 on both SMAs. The land patterns are near-identical,
so the swap cost almost nothing in routing:

                     Amphenol 132289      Linx CONSMA020.062-G
  ground pitch       +/-4.250             +/-4.26
  centre pad         1.50 x 5.08          1.50 x 5.60
  ground pads        1.50 x 5.08, F+B     1.60 x 4.90, F+B
  voltage rating     not published        500 V RMS

The voltage rating is the reason this matters. J1 carries HV_OUT and HV_RAIL at
~250 V, and the Amphenol part has no published rating -- a gap inherited from
upstream. 500 V RMS from TE's Table I closes it. Also 50 ohm, DC-18 GHz,
-65 to +165 C, 5000 Mohm insulation resistance.

New footprint picoemp:SMA_Linx_CONSMA020_062_G_EdgeMount, land pattern taken
from sheet 2 of ENG_DS_L9000279-01_A. Its origin is the BOARD EDGE with +X
into the board, which suits an edge launch far better than the stock Amphenol
convention of origin-at-centre-pad. Copper is set back 0.100 mm from that
origin: pads flush to the edge overlap the Edge.Cuts graphic and DRC flags them
even under the existing 0 mm edge exception. The Amphenol footprint does the
same thing with 0.090 mm.

Placement: J1 (124.390,175.272) rot 90, J4 (137.400,45.272) rot -90 -- origins
sitting on Edge.Cuts. Pads land within 0.01 mm of where the Amphenol's were, so
no track moved.

tools/prepare_linx_sma_model.py re-axes TE's L9000279-01.STEP into KiCad's
frame: model X = STEP Z + 4.700, Y = STEP X, Z = STEP Y - 0.785, putting the
flange face on the board edge and the connector axis at mid-thickness of a
1.57 mm board. Determinant +1, so it rotates rather than mirrors. The STEP is
gitignored like the Hammond models -- fetch the vendor zip and re-run the tool.

Schematic updated: MPN, Manufacturer, DigiKey, Datasheet and Footprint on both
J1 and J4. tests/test_schematic.py's FOOTPRINTS dict updated to match.

Zones refilled -- the longer centre pad initially collide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
Parts:
- J1, J4: footprint Connector_Coaxial:SMA_Amphenol_132289_EdgeMount -> picoemp:SMA_Linx_CONSMA020_062_G_EdgeMount; DigiKey (none) -> 343-CONSMA020.062-G-ND; MPN 132289 -> CONSMA020.062-G; Manufacturer Amphenol -> TE Connectivity Linx
Changed lines of the file:
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@@
 			)
 		)
-		(property "Footprint" "Connector_Coaxial:SMA_Amphenol_132289_EdgeMount"
+		(property "Footprint" "picoemp:SMA_Linx_CONSMA020_062_G_EdgeMount"
 			(at 313.69 92.71 0)
 			(hide yes)
@@
 			)
 		)
-		(property "Datasheet" ""
+		(property "Datasheet" "https://www.te.com/usa-en/product-CONSMA020.062-G.html"
 			(at 313.69 92.71 0)
 			(hide yes)
@@
 			)
 		)
-		(property "Manufacturer" "Amphenol"
+		(property "Manufacturer" "TE Connectivity Linx"
 			(at -136.31 12.71 0)
 			(hide yes)
@@
 			)
 		)
-		(property "MPN" "132289"
+		(property "MPN" "CONSMA020.062-G"
 			(at -136.31 12.71 0)
 			(hide yes)
@@
 					(size 1.27 1.27)
 				)
+			)
+		)
+		(property "DigiKey" "343-CONSMA020.062-G-ND" (at 0 0 0)
+			(effects
+				(font
+					(size 1.27 1.27)
+				)
+				(hide yes)
 			)
 		)
@@
 			)
 		)
-		(property "Footprint" "Connector_Coaxial:SMA_Amphenol_132289_EdgeMount"
+		(property "Footprint" "picoemp:SMA_Linx_CONSMA020_062_G_EdgeMount"
 			(at 420.37 276.86 0)
 			(hide yes)
@@
 			)
 		)
-		(property "Datasheet" ""
+		(property "Datasheet" "https://www.te.com/usa-en/product-CONSMA020.062-G.html"
 			(at 420.37 276.86 0)
 			(hide yes)
@@
 			)
 		)
-		(property "Manufacturer" "Amphenol"
+		(property "Manufacturer" "TE Connectivity Linx"
 			(at 0 0 0)
 			(hide yes)
@@
 			)
 		)
-		(property "MPN" "132289"
+		(property "MPN" "CONSMA020.062-G"
 			(at 0 0 0)
 			(hide yes)
@@
 			)
 		)
+		(property "DigiKey" "343-CONSMA020.062-G-ND" (at 0 0 0)
+			(effects
+				(font
+					(size 1.27 1.27)
+				)
+				(hide yes)
+			)
+		)

Commit message: C3: Murata KRM55 metal-terminal part -> TDK CGA9P1X7T2J474K250KE
The Murata part was a package mismatch. KRM is Murata's Metal Terminal Type:
KRM55TR72J474MH01K is a two-chip stack on a J-lead frame, 6.1 x 5.3 x 4.80 mm,
and Murata's own test jig wants pads 2.6 x 8.0 on a 5.6 mm gap. The board has
Capacitor_SMD:C_2220_5750Metric -- pads 1.8 x 5.4 at +/-2.55. The J-leads did
land on that (feet at +/-1.85..3.05 inside pads at +/-1.65..3.45) but with only
0.05 mm of pad either side across the width, against 1.35 mm in Murata's jig.
Poor fillet support for a 4.8 mm tall two-chip part on the highest-energy node
on the board.

TDK CGA9P1X7T2J474K250KE is a plain 2220 chip: 0.47 uF +/-10%, 630 V, X7T,
5.7 x 5.0 x 2.80 mm, soft termination, AEC-Q200, -55 to +125 C. DigiKey
445-8764-1-ND, 7555 in stock.

  no board change -- C_2220_5750Metric is the correct land for it
  2.80 mm not 4.80, so it clears upstream's "must be below 5 mm to fit shield"
      by 2.2 mm instead of 0.2, and the 2.90 mm KiCad 3D model is now honest
      rather than understating the part by 1.9 mm
  X7T is what the schematic Value has always said -- that field was right and
      the Murata MPN was the odd one out
  soft termination matters on a 2220 sitting near a board edge between two
      mounting holes; flex cracking is the failure mode for that case size
  +/-10% rather than +/-20%

Gates: 66 tests pass; ERC exit 0; DRC --severity-error exit 0; DRC with
warnings 0 violations, 0 unconnected, 0 footprint errors -- the three fiducial
DNP warnings have also gone, cleared by the silkscreen work.

bom/ regenerated.

Co-Authored-By: Claude Opus 5 <noreply@anthropic.com>
Parts:
- C3: DigiKey 490-16845-1-ND -> 445-8764-1-ND; MPN KRM55TR72J474MH01K -> CGA9P1X7T2J474K250KE; Manufacturer Murata -> TDK
Changed lines of the file:
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@@
 			)
 		)
-		(property "Datasheet" ""
+		(property "Datasheet" "https://product.tdk.com/en/search/capacitor/ceramic/mlcc/info?part_no=CGA9P1X7T2J474K250KE"
 			(at 345.44 284.48 0)
 			(hide yes)
@@
 			)
 		)
-		(property "DigiKey" "490-16845-1-ND"
+		(property "DigiKey" "445-8764-1-ND"
 			(at 0 0 0)
 			(hide yes)
@@
 			)
 		)
-		(property "Manufacturer" "Murata"
+		(property "Manufacturer" "TDK"
 			(at 0 0 0)
 			(hide yes)
@@
 			)
 		)
-		(property "MPN" "KRM55TR72J474MH01K"
+		(property "MPN" "CGA9P1X7T2J474K250KE"
 			(at 0 0 0)
 			(hide yes)

Commit message: J3: MKDS -> MKDSN 1,5/2-5,08 for 630 V headroom, with a local footprint
J3 sits across HV_SENSE/HV_RTN at ~246 V on a 300 V-rated MKDS. Phoenix
publishes the MKDSN's rating per IEC 60664-1 category rather than as one number:

  III/3   250 V   clearance 3 mm   creepage 3.2 mm
  III/2   400 V   clearance 3 mm   creepage 3.0 mm
  II/2    630 V   clearance 3 mm   creepage 3.2 mm

This board is USB-powered, mains-isolated and enclosed, which is overvoltage
category II / pollution degree 2 -- so 630 V applies, giving 2.6x margin and
clearing upstream's 400 V barrier design rating. Material group I, CTI 600,
4 kV rated surge, UL94 V0, glow wire 850 C. cULus recognition is 300 V / 10 A
and VDE 400 V / 17.5 A, which are the numbers to quote if a listing is ever
needed.

Chose MKDSN (0 deg entry) over SMKDSN (45 deg). They are electrically
identical; the MKDSN is 10.16 x 8.15 x 13.5 against the SMKDSN's
11.16 x 12 x 14.5. The SMKDSN is larger than the existing courtyard in both
axes and leaves only 0.55 mm under the 1551G shield, versus 1.55 mm for the
MKDSN -- itself better than the 1.25 mm the MKDS had.

New picoemp:TerminalBlock_Phoenix_MKDSN-1,5-2-5.08_1x02_P5.08mm_Horizontal.
Copper is unchanged from the stock MKDS land -- 1.3 mm drill, 2.6 mm pad,
5.08 pitch -- so the pads landed on exactly the same coordinates and nothing
rerouted. Only the outline differs: 8.15 deep rather than 9.8. The datasheet
does not publish where the pins sit within that depth, so the outline keeps the
rear edge where the MKDS had it and pulls the front in by 1.65 mm; that is silk
and courtyard only, noted in the footprint description.

Also corrected J3's schematic Description to carry the real ratings, and
replaced the BOM comment that still claimed a milled slot between the pads --
that slot was never cut, and the 5.08 mm part's 2.480 mm pad separation is the
documented fallback.

DigiKey PN cleared -- the MKDSN needs looking up. bom/ regenerated and J3 now
shows the Phoenix item number 1548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
Parts:
- J3: value MKDS 1,5/2-5.08 -> MKDSN 1,5/2-5,08; footprint TerminalBlock_Phoenix:TerminalBlock_Phoenix_MKDS-1,5-2-5.08_1x02_P5.08mm_Horizontal -> picoemp:TerminalBlock_Phoenix_MKDSN-1,5-2-5.08_1x02_P5.08mm_Horizontal; BOM Comments HV calibration tap. Milled slot between pads - see spec sec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 -> HV calibration tap, optional -- upstream fits it only for c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; DigiKey 277-1263-ND -> (none); MPN 1715721 -> 1548128
Changed lines of the file:
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@@
 			)
 		)
-		(property "Value" "MKDS 1,5/2-5.08"
+		(property "Value" "MKDSN 1,5/2-5,08"
 			(at 387.35 218.4399 0)
 			(show_name no)
@@
 			)
 		)
-		(property "Footprint" "TerminalBlock_Phoenix:TerminalBlock_Phoenix_MKDS-1,5-2-5.08_1x02_P5.08mm_Horizontal"
+		(property "Footprint" "picoemp:TerminalBlock_Phoenix_MKDSN-1,5-2-5.08_1x02_P5.08mm_Horizontal"
 			(at 386.08 215.9 0)
 			(hide yes)
@@
 			)
 		)
-		(property "Datasheet" ""
+		(property "Datasheet" "https://www.phoenixcontact.com/us/products/1548128"
 			(at 386.08 215.9 0)
 			(hide yes)
@@
 			)
 		)
-		(property "Description" "HV calibration tap, 5.08mm pitch PCB terminal block, replaces BG306 (2.07mm pad gap failed IEC 60664-1 creepage at ~600V)"
+		(property "Description" "HV calibration tap, 5.08mm pitch PCB terminal block. 630 V at IEC 60664-1 II/2 (400 V III/2, 250 V III/3), CTI 600, creepage 3.2mm. Replaced MKDS 1,5/2-5.08 (300 V) for headroom on a ~246V node; MKDS replaced BG306 whose 2.07mm pad gap failed creepage."
 			(at 386.08 215.9 0)
 			(hide yes)
@@
 			)
 		)
-		(property "MPN" "1715721"
+		(property "MPN" "1548128"
 			(at 0 0 0)
 			(hide yes)
@@
 			)
 		)
-		(property "DigiKey" "277-1263-ND"
+		(property "DigiKey" ""
 			(at 0 0 0)
 			(hide yes)
@@
 			)
 		)
-		(property "BOM Comments" "HV calibration tap. Milled slot between pads - see spec section 7.3."
+		(property "BOM Comments" "HV calibration tap, optional -- upstream fits it only for charge-voltage calibration. Drop-in on the MKDS land: same 1.3mm drill and 5.08 pitch."
 			(at 0 0 0)
 			(hide yes)

Commit message: C3: TDK CGA9P -> Murata GR355DD7LQ474KW01K on cost
Same electricals -- 0.47 uF +/-10%, 630 V, X7T, 2220, -55 to +125 C, and the
same +22/-33% capacitance change over range. Both are plain chips that fit
C_2220_5750Metric with no board change. $1.237 against $4.50, so 3.6x cheaper.

What the TDK had over it was soft termination and AEC-Q200. Soft termination is
worth having here in principle: C3 is a 2220 sitting 9.9 mm from MH2, and
tightening that screw flexes the board right beside it, which is the classic way
to crack a 2220. But at 3.6x the price the better hedge for a five-board hand-
built run is to buy spares and be careful with the screw, rather than pay for
soft termination on every piece. AEC-Q200 buys nothing on a bench instrument.

The Murata is also 2.0 mm thick against the TDK's 2.80. Marginally helpful --
a thinner chip is slightly less prone to flex cracking, and the KiCad 2220 3D
model at 2.90 mm now overstates rather than understates the part.

Discounted its "high ripple current" billing: that targets continuous SMPS
ripple, whereas this is a ~15 mJ single-shot discharge at low repetition rate,
which any 630 V 2220 handles.

Assembly note recorded in C3's BOM comment: buy spares, go gentle on MH2.

Gates: 66 tests pass; ERC exit 0; DRC exit 0 with warnings included.
bom/ regenerated.

Co-Authored-By: Claude Opus 5 <noreply@anthropic.com>
Parts:
- C3: BOM Comments (none) -> HV storage cap, 5.7x5.0x2.0 plain chip on C_2220_5750Metric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; DigiKey 445-8764-1-ND -> 490-GR355DD7LQ474KW01KCT-ND; MPN CGA9P1X7T2J474K250KE -> GR355DD7LQ474KW01K; Manufacturer TDK -> Murata Electronics
Changed lines of the file:
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@@
 			)
 		)
-		(property "Datasheet" "https://product.tdk.com/en/search/capacitor/ceramic/mlcc/info?part_no=CGA9P1X7T2J474K250KE"
+		(property "Datasheet" "https://search.murata.co.jp/Ceramy/image/img/A01X/G101/ENG/GR355DD7LQ474KW01-01.pdf"
 			(at 345.44 284.48 0)
 			(hide yes)
@@
 			)
 		)
-		(property "DigiKey" "445-8764-1-ND"
+		(property "DigiKey" "490-GR355DD7LQ474KW01KCT-ND"
 			(at 0 0 0)
 			(hide yes)
@@
 			)
 		)
-		(property "Manufacturer" "TDK"
+		(property "Manufacturer" "Murata Electronics"
 			(at 0 0 0)
 			(hide yes)
@@
 			)
 		)
-		(property "MPN" "CGA9P1X7T2J474K250KE"
+		(property "MPN" "GR355DD7LQ474KW01K"
 			(at 0 0 0)
 			(hide yes)
@@
 			)
 		)
+		(property "BOM Comments" "HV storage cap, 5.7x5.0x2.0 plain chip on C_2220_5750Metric. Buy spares -- no soft termination, and MH2 is 9.9mm away, so go gentle tightening that screw." (at 0 0 0)
+			(effects
+				(font
+					(size 1.27 1.27)
+				)
+				(hide yes)
+			)
+		)
