File: hardware/rev2026/picoemp-rev2026.kicad_sch (KiCad schematic)
At the start: 53 parts, among them J1 EDGE-SMA, J2 1x2_Pin_Header, J3 MKDSN 1,5/2-5,08, J4 EDGE-SMA, P1 Header 7, P2 Header 2, P3 Header 4, Q1 LDA111STR, Q2 RGT16BM65DTL, Q3 AO3422, Q4 AO3422, SW1 KSC741J LFS, SW2 KSC741J LFS, SW3 TL3301AF160QJ, T1 ATB322524, T2 ATB322524, U1 SC0915, U2 74LVC1G17

Commit message: Rev B board: re-designate the schematic against the PCB, arm switch to GND
All gates green: ERC 0 violations, DRC 0 violations / 0 unconnected /
0 schematic parity issues, 85 tests passing.

The schematic had been re-annotated with reset, which renumbers every
symbol sequentially and destroys correspondence with the PCB. The
signature was the gaps closing up -- the schematic had C1-C5 and R1-R15
with no gaps against the PCB's C1,C2,C3,C5,C6 and R1-R7,R9-R16. 38
components ended up on the wrong designator, including the IGBT labelled
Q4, the 630 V storage cap labelled C4, and the 20 M HV sense resistor
labelled R12.

Repaired from UUIDs rather than by inference. Every PCB footprint stores
(path "/uuid") pointing at its schematic symbol and annotation does not
touch UUIDs, so the true mapping survived: 52 footprints, 52 matches,
no orphans, one bijection. Each symbol's Reference property and its
instances reference were rewritten from it.

Note that --schematic-parity reported 0 issues throughout, while the
design was fully scrambled. It is not a safety net for this failure mode.

Roles that moved with the rev: the HV terminal block J3 -> J4, the
trigger SMA J4 -> J3, and the three headers P1/P2/P3 consolidated into a
5-pin J5 and a 7-pin J6. Tests follow the part, not the designator.

The arm switch now pulls to GND rather than up to 3V3, so both switches
are active-low against an internal pullup. cspico_simple.py and
bringup.py updated to match; the fault-injection path is unchanged.

BRINGUP-LOG.md gains a header mapping board #1's designators to rev B's
by function, and records that the current bringup.py will fail the ARM
check on board #1, whose arm switch drives high.

Stale generated output deliberately not committed: the gerbers under
production/ are from 19:56 and ibom.html from 14:40, against a board
saved at 23:00. Regenerate before ordering.

Co-Authored-By: Claude Opus 5 <noreply@anthropic.com>
Parts:
- removed P2: Header 2, Connector_PinHeader_2.54mm:PinHeader_1x02_P2.54mm_Vertical, symbol Connector:Conn_01x02_Pin
- C1, C2, C3, C5, C6, D6, D8, D9, R1, R10, R11, R12, R13, R14, R15, R16, R2, R3, R4, R5, R6, R7, R9: KiLib_Generator (none) -> SMD_2terminal_chip_molded
- FID1, FID2, FID3: KiLib_Generator (none) -> fiducial
- J2: KiLib_Generator (none) -> connector/JST
- J5: renamed from P3; footprint Connector_PinHeader_2.54mm:PinHeader_1x04_P2.54mm_Vertical -> Connector_PinHeader_2.54mm:PinHeader_1x05_P2.54mm_Vertical; symbol Connector:Conn_01x04_Pin -> Connector:Conn_01x05_Pin; KiLib_Generator (none) -> connector/pin_header_socket
- J6: renamed from P1; KiLib_Generator (none) -> connector/pin_header_socket
- MH1, MH2, MH3: KiLib_Generator (none) -> mounting_hardware/mounting_hole
- Q2: KiLib_Generator (none) -> package/TO_SOT/SMD
- Q3, Q4, U2: KiLib_Generator (none) -> package/gullwing
- renumbered J4 to J3, J3 to J4
Connections:
- net +3V3: now also J5.1 (Pin_1); no longer J5.2 (Pin_2), SW1.2
- net CHARGED: now also J5.2 (Pin_2); no longer J5.1 (Pin_1)
- net GND: now also J5.5 (Pin_5), SW1.2; no longer J5.3 (Pin_3)
- net HVPULSE: now also J5.3 (Pin_3)
Other:
- note removed: "Physical"
- moved on the sheet: MH1, MH2, MH3
