File: hardware/rev2026/picoemp-rev2026.kicad_pcb (KiCad board)
At the start: 2 copper layers, 40 x 130 mm, 53 parts, among them J1 EDGE-SMA, J2 1x2_Pin_Header, J3 MKDSN 1,5/2-5,08, J4 EDGE-SMA, P1 Header 7, P2 Header 2, P3 Header 4, Q1 LDA111STR, Q2 RGT16BM65DTL, Q3 AO3422, Q4 AO3422, SW1 KSC741J LFS, SW2 KSC741J LFS, SW3 TL3301AF160QJ, T1 ATB322524, T2 ATB322524, U1 SC0915, U2 74LVC1G17

Commit message: Rev B board: re-designate the schematic against the PCB, arm switch to GND
All gates green: ERC 0 violations, DRC 0 violations / 0 unconnected /
0 schematic parity issues, 85 tests passing.

The schematic had been re-annotated with reset, which renumbers every
symbol sequentially and destroys correspondence with the PCB. The
signature was the gaps closing up -- the schematic had C1-C5 and R1-R15
with no gaps against the PCB's C1,C2,C3,C5,C6 and R1-R7,R9-R16. 38
components ended up on the wrong designator, including the IGBT labelled
Q4, the 630 V storage cap labelled C4, and the 20 M HV sense resistor
labelled R12.

Repaired from UUIDs rather than by inference. Every PCB footprint stores
(path "/uuid") pointing at its schematic symbol and annotation does not
touch UUIDs, so the true mapping survived: 52 footprints, 52 matches,
no orphans, one bijection. Each symbol's Reference property and its
instances reference were rewritten from it.

Note that --schematic-parity reported 0 issues throughout, while the
design was fully scrambled. It is not a safety net for this failure mode.

Roles that moved with the rev: the HV terminal block J3 -> J4, the
trigger SMA J4 -> J3, and the three headers P1/P2/P3 consolidated into a
5-pin J5 and a 7-pin J6. Tests follow the part, not the designator.

The arm switch now pulls to GND rather than up to 3V3, so both switches
are active-low against an internal pullup. cspico_simple.py and
bringup.py updated to match; the fault-injection path is unchanged.

BRINGUP-LOG.md gains a header mapping board #1's designators to rev B's
by function, and records that the current bringup.py will fail the ARM
check on board #1, whose arm switch drives high.

Stale generated output deliberately not committed: the gerbers under
production/ are from 19:56 and ibom.html from 14:40, against a board
saved at 23:00. Regenerate before ordering.

Co-Authored-By: Claude Opus 5 <noreply@anthropic.com>
Parts:
- removed P2: Header 2, Connector_PinHeader_2.54mm:PinHeader_1x02_P2.54mm_Vertical
- J5: renamed from P3; footprint Connector_PinHeader_2.54mm:PinHeader_1x04_P2.54mm_Vertical -> Connector_PinHeader_2.54mm:PinHeader_1x05_P2.54mm_Vertical
- moved SW2 6.50 mm to (108.7, 102.8)
- moved J5 5.22 mm to (119.3, 118.7)
- moved D8 1.81 mm to (107.9, 86.3)
- moved R12 1.80 mm to (111.1, 86.3)
- moved SW1 1.15 mm to (140.0, 76.0)
- moved D2 0.72 mm to (130.8, 142.7)
- moved J2 0.55 mm to (133.9, 57.1)
- moved J3 0.43 mm to (137.4, 45.7)
- moved D6 0.21 mm to (107.9, 82.8)
- moved C2 0.20 mm to (131.4, 133.4)
- moved D9 0.12 mm to (141.7, 83.2)
- renumbered J4 to J3, J3 to J4, P1 to J6
Connections:
- J5 pad 1: /CHARGED -> +3V3
- J5 pad 2: +3V3 -> /CHARGED
- J5 pad 3: GND -> /HVPULSE
- SW1 pad 2: +3V3 -> GND
Routing:
- net +3V3: track 102.9 -> 96.4 mm, vias 2 -> 4
- net /CHARGED: track 61.7 -> 57.3 mm, vias 0 -> 1
- net /HV_RAIL: track 43.5 -> 39.4 mm
- net GND: track 63.6 -> 60.7 mm, vias 94 -> 98
- net /HVPWM: track 30.1 -> 32.8 mm, vias 0 -> 1
- net /HVPULSE: track 24.2 -> 21.8 mm, vias 0 -> 1
- net /HV_RTN: track 90.7 -> 92.3 mm
- net /STATUS_LED: track 2.94 -> 3.58 mm
- net /T2_PRI_B: track 4.19 -> 3.64 mm
- net /HV_RECT: track 4.19 -> 3.64 mm
Other:
- board text added: "HIGH VOLT"
- board text added: "PicoEMP 2026 Alex Gompper Rev B 28.7.2026"
- board text removed: "+3V3"
- board text removed: "CHARGED"
- board text removed: "H.V."
- board text removed: "HVPULSE"
- board text removed: "HVPWM"
- board text removed: "PicoEMP 2026 Alex Gompper Rev A 28.7.2026"
